Commit message: Update rover URDF to version 2 with adjustments
Updated rover URDF file to version 2 with changes in wheel positioning, track collision properties, and friction coefficients.

File: urdf/rover.urdf.xacro (robot description, xacro)
@@ -2,14 +2,12 @@
 <robot name="lunar_rover" xmlns:xacro="http://www.ros.org/wiki/xacro">
   <!-- ============================================================
-       ROVER LUNAR TMR 2026
-       Chasis: 27cm x 20.5cm x 10cm  (orugas diferenciales)
-       Brazo:  6 DOF (MG996R x3 + MG90S x3)
-         - a = 9.5cm  base
-         - b = 11.5cm upper arm
-         - c = 10cm   forearm
-         - d = 3cm    wrist_pitch
-         - e = 7cm    wrist_roll + gripper
-       ============================================================ -->
-  <!-- Propiedades globales -->
+       ROVER LUNAR TMR 2026 — URDF v2 (física estable)
+       Cambios vs v1:
+       1. Ruedas reposicionadas (no penetran el suelo)
+       2. Orugas son SOLO visuales (sin collision)
+       3. Fricción reducida (mu=0.8 en vez de 1.5)
+       4. kp reducido (100000 en vez de 500000)
+       5. max_wheel_acceleration bajado (3.0 en vez de 10.0)
+       ============================================================ -->
   <xacro:property name="PI" value="3.14159265"/>
   <!-- Chasis -->
@@ -17,6 +15,10 @@
   <xacro:property name="chassis_width"  value="0.205"/>
   <xacro:property name="chassis_height" value="0.10"/>
-  <xacro:property name="chassis_mass"   value="3.0"/>
-  <!-- Orugas (representadas como cajas planas) -->
+  <xacro:property name="chassis_mass"   value="3.5"/>
+  <!-- Ruedas motrices -->
+  <xacro:property name="wheel_radius"   value="0.0575"/>
+  <xacro:property name="wheel_width"    value="0.04"/>
+  <xacro:property name="wheel_mass"     value="0.2"/>
+  <!-- Orugas (SOLO VISUALES ahora) -->
   <xacro:property name="track_length"   value="0.27"/>
   <xacro:property name="track_width"    value="0.04"/>
@@ -24,26 +26,14 @@
   <xacro:property name="track_offset_y" value="0.1225"/>
   <!-- Brazo -->
-  <xacro:property name="base_h"     value="0.095"/>   <!-- a -->
-  <xacro:property name="upper_l"    value="0.115"/>   <!-- b -->
-  <xacro:property name="forearm_l"  value="0.100"/>   <!-- c -->
-  <xacro:property name="wrist_p_l"  value="0.030"/>   <!-- d -->
-  <xacro:property name="wrist_r_l"  value="0.040"/>   <!-- e/2 -->
-  <xacro:property name="gripper_l"  value="0.030"/>   <!-- e/2 -->
-  <!-- Colores Gazebo -->
-  <material name="dark_grey">
-    <color rgba="0.2 0.2 0.2 1"/>
-  </material>
-  <material name="light_grey">
-    <color rgba="0.6 0.6 0.6 1"/>
-  </material>
-  <material name="black">
-    <color rgba="0.05 0.05 0.05 1"/>
-  </material>
-  <material name="orange">
-    <color rgba="1.0 0.5 0.0 1"/>
-  </material>
-  <!-- ============================================================
-       MACRO: Inercia de caja
-       ============================================================ -->
+  <xacro:property name="base_h"     value="0.095"/>
+  <xacro:property name="upper_l"    value="0.115"/>
+  <xacro:property name="forearm_l"  value="0.100"/>
+  <xacro:property name="wrist_p_l"  value="0.030"/>
+  <xacro:property name="wrist_r_l"  value="0.040"/>
+  <xacro:property name="gripper_l"  value="0.030"/>
+  <material name="dark_grey"><color rgba="0.2 0.2 0.2 1"/></material>
+  <material name="light_grey"><color rgba="0.6 0.6 0.6 1"/></material>
+  <material name="black"><color rgba="0.05 0.05 0.05 1"/></material>
+  <material name="orange"><color rgba="1.0 0.5 0.0 1"/></material>
   <xacro:macro name="box_inertia" params="m x y z">
     <inertial>
@@ -63,5 +53,7 @@
   </xacro:macro>
   <!-- ============================================================
-       BASE LINK (referencia del robot)
+       BASE LINKS
+       base_footprint = referencia en el suelo (z=0)
+       base_link = chasis, elevado UN RADIO DE RUEDA sobre el suelo
        ============================================================ -->
   <link name="base_footprint"/>
@@ -69,5 +61,6 @@
     <parent link="base_footprint"/>
     <child link="base_link"/>
-    <origin xyz="0 0 ${track_height/2}" rpy="0 0 0"/>
+    <!-- base_link a la altura del centro de las ruedas -->
+    <origin xyz="0 0 ${wheel_radius}" rpy="0 0 0"/>
   </joint>
   <!-- ============================================================
@@ -94,5 +87,6 @@
   </link>
   <!-- ============================================================
-       ORUGAS — izquierda y derecha (visuales + colisión)
+       ORUGAS — SOLO VISUALES (sin collision)
+       Las "tracks" solo decoran. Las ruedas hacen el trabajo físico.
        ============================================================ -->
   <xacro:macro name="track" params="side reflect">
@@ -105,17 +99,17 @@
         <material name="black"/>
       </visual>
-      <collision>
-        <origin xyz="0 0 0" rpy="0 0 0"/>
-        <geometry>
-          <box size="${track_length} ${track_width} ${track_height}"/>
-        </geometry>
-      </collision>
-      <xacro:box_inertia m="0.3" x="${track_length}" y="${track_width}" z="${track_height}"/>
+      <!-- NO collision aquí — orugas son visuales nomas -->
+      <inertial>
+        <mass value="0.05"/>
+        <inertia ixx="0.0001" ixy="0" ixz="0"
+                 iyy="0.0001" iyz="0"
+                 izz="0.0001"/>
+      </inertial>
     </link>
     <joint name="track_${side}_joint" type="fixed">
       <parent link="base_link"/>
       <child link="track_${side}"/>
-      <origin xyz="0 ${reflect*track_offset_y} ${-(chassis_height/2 - track_height/2 + 0.005)}"
-              rpy="0 0 0"/>
+      <!-- Centrada vertical respecto al chasis -->
+      <origin xyz="0 ${reflect*track_offset_y} -0.0075" rpy="0 0 0"/>
     </joint>
   </xacro:macro>
@@ -123,6 +117,7 @@
   <xacro:track side="right" reflect="-1"/>
   <!-- ============================================================
-       RUEDAS MOTRICES — izquierda y derecha (para differential drive)
-       Gazebo las usa internamente para calcular movimiento
+       RUEDAS MOTRICES — únicos contactos con el suelo
+       Centro de rueda a la altura de base_link (z=wheel_radius absoluto)
+       Esto asegura que la rueda toque el suelo PERFECTAMENTE.
        ============================================================ -->
   <xacro:macro name="drive_wheel" params="side reflect">
@@ -131,5 +126,5 @@
         <origin xyz="0 0 0" rpy="${PI/2} 0 0"/>
         <geometry>
-          <cylinder radius="0.0575" length="0.04"/>
+          <cylinder radius="${wheel_radius}" length="${wheel_width}"/>
         </geometry>
         <material name="black"/>
@@ -138,16 +133,17 @@
         <origin xyz="0 0 0" rpy="${PI/2} 0 0"/>
         <geometry>
-          <cylinder radius="0.0575" length="0.04"/>
+          <cylinder radius="${wheel_radius}" length="${wheel_width}"/>
         </geometry>
       </collision>
-      <xacro:cylinder_inertia m="0.2" r="0.0575" h="0.04"/>
+      <xacro:cylinder_inertia m="${wheel_mass}" r="${wheel_radius}" h="${wheel_width}"/>
     </link>
     <joint name="wheel_${side}_joint" type="continuous">
       <parent link="base_link"/>
       <child link="wheel_${side}"/>
-      <origin xyz="0 ${reflect*(chassis_width/2 + 0.02)} ${-chassis_height/2 + 0.005}"
-              rpy="0 0 0"/>
+      <!-- z=0: centro de la rueda en la misma altura que base_link -->
+      <!-- y: ligeramente fuera del chasis para que las orugas las cubran -->
+      <origin xyz="0 ${reflect*(chassis_width/2 + 0.02)} 0" rpy="0 0 0"/>
       <axis xyz="0 1 0"/>
-      <dynamics damping="0.1" friction="0.5"/>
+      <dynamics damping="0.05" friction="0.1"/>
     </joint>
   </xacro:macro>
@@ -156,5 +152,4 @@
   <!-- ============================================================
        SENSOR LIDAR — LD14P
-       Montado encima del chasis, al frente-centro
        ============================================================ -->
   <link name="lidar_link">
@@ -180,5 +175,5 @@
   </joint>
   <!-- ============================================================
-       CÁMARA RGB-D — AstraPro (frontal)
+       CÁMARA RGB-D — AstraPro
        ============================================================ -->
   <link name="camera_link">
@@ -200,5 +195,6 @@
     <parent link="base_link"/>
     <child link="camera_link"/>
-    <origin xyz="${chassis_length/2 - 0.01} 0 ${chassis_height/2 + 0.015}" rpy="0 0.2 0"/>
+    <!-- Inclinación reducida a 0.1 rad (5.7 grados) — más estable visualmente -->
+    <origin xyz="${chassis_length/2 - 0.01} 0 ${chassis_height/2 + 0.015}" rpy="0 0.1 0"/>
   </joint>
   <link name="camera_optical_link"/>
@@ -209,8 +205,6 @@
   </joint>
   <!-- ============================================================
-       BRAZO ROBÓTICO — 6 DOF (diseño propio)
-       Montado en la parte trasera-centro del chasis
-       ============================================================ -->
-  <!-- --- LINK 0: Base fija del brazo sobre el chasis --- -->
+       BRAZO ROBÓTICO — 6 DOF
+       ============================================================ -->
   <link name="arm_base_link">
     <visual>
@@ -234,5 +228,4 @@
     <origin xyz="${-chassis_length/2 + 0.08} 0 ${chassis_height/2}" rpy="0 0 0"/>
   </joint>
-  <!-- --- JOINT 1: Rotación base (yaw) — MG996R --- -->
   <joint name="joint_1" type="revolute">
     <parent link="arm_base_link"/>
@@ -243,5 +236,4 @@
     <dynamics damping="0.05" friction="0.1"/>
   </joint>
-  <!-- --- LINK 1: Hombro (upper arm b=11.5cm) --- -->
   <link name="link_1">
     <visual>
@@ -260,5 +252,4 @@
     <xacro:box_inertia m="0.15" x="0.04" y="0.04" z="${upper_l}"/>
   </link>
-  <!-- --- JOINT 2: Hombro (pitch) — MG996R --- -->
   <joint name="joint_2" type="revolute">
     <parent link="link_1"/>
@@ -269,5 +260,4 @@
     <dynamics damping="0.05" friction="0.1"/>
   </joint>
-  <!-- --- LINK 2: Codo (forearm c=10cm) --- -->
   <link name="link_2">
     <visual>
@@ -286,5 +276,4 @@
     <xacro:box_inertia m="0.12" x="${forearm_l}" y="0.035" z="0.035"/>
   </link>
-  <!-- --- JOINT 3: Codo (pitch) — MG996R --- -->
   <joint name="joint_3" type="revolute">
     <parent link="link_2"/>
@@ -295,5 +284,4 @@
     <dynamics damping="0.05" friction="0.1"/>
   </joint>
-  <!-- --- LINK 3: Muñeca pitch (d=3cm) --- -->
   <link name="link_3">
     <visual>
@@ -312,5 +300,4 @@
     <xacro:box_inertia m="0.05" x="${wrist_p_l}" y="0.03" z="0.03"/>
   </link>
-  <!-- --- JOINT 4: Muñeca pitch — MG90S --- -->
   <joint name="joint_4" type="revolute">
     <parent link="link_3"/>
@@ -321,5 +308,4 @@
     <dynamics damping="0.02" friction="0.05"/>
   </joint>
-  <!-- --- LINK 4: Muñeca roll --- -->
   <link name="link_4">
     <visual>
@@ -338,5 +324,4 @@
     <xacro:cylinder_inertia m="0.04" r="0.018" h="${wrist_r_l}"/>
   </link>
-  <!-- --- JOINT 5: Muñeca roll — MG90S --- -->
   <joint name="joint_5" type="revolute">
     <parent link="link_4"/>
@@ -347,5 +332,4 @@
     <dynamics damping="0.02" friction="0.05"/>
   </joint>
-  <!-- --- LINK 5: Conector gripper --- -->
   <link name="link_5">
     <visual>
@@ -364,5 +348,4 @@
     <xacro:box_inertia m="0.03" x="${gripper_l}" y="0.04" z="0.025"/>
   </link>
-  <!-- --- JOINT 6: Apertura del gripper — MG90S --- -->
   <joint name="joint_6" type="revolute">
     <parent link="link_5"/>
@@ -373,5 +356,4 @@
     <dynamics damping="0.01" friction="0.02"/>
   </joint>
-  <!-- --- LINK GRIPPER --- -->
   <link name="gripper_link">
     <visual>
@@ -390,5 +372,4 @@
     <xacro:box_inertia m="0.015" x="0.04" y="0.008" z="0.02"/>
   </link>
-  <!-- Frame del efector final (tool center point) -->
   <link name="tcp_link"/>
   <joint name="tcp_joint" type="fixed">
@@ -398,19 +379,17 @@
   </joint>
   <!-- ============================================================
-       PLUGINS DE GAZEBO
-       ============================================================ -->
-  <!-- Plugin differential drive (simula movimiento de orugas) -->
+       PLUGINS GAZEBO
+       ============================================================ -->
+  <!-- Diff drive: aceleración reducida a 3.0 m/s2 (era 10.0) -->
   <gazebo>
     <plugin name="differential_drive_controller"
             filename="libgazebo_ros_diff_drive.so">
-      <ros>
-        <namespace>/rover</namespace>
-      </ros>
+      <ros><namespace>/rover</namespace></ros>
       <left_joint>wheel_left_joint</left_joint>
       <right_joint>wheel_right_joint</right_joint>
-      <wheel_separation>${chassis_width + 0.04}</wheel_separation>
+      <wheel_separation>0.245</wheel_separation>
       <wheel_diameter>0.115</wheel_diameter>
       <max_wheel_torque>20</max_wheel_torque>
-      <max_wheel_acceleration>10.0</max_wheel_acceleration>
+      <max_wheel_acceleration>3.0</max_wheel_acceleration>
       <command_topic>cmd_vel</command_topic>
       <publish_odom>true</publish_odom>
@@ -422,5 +401,5 @@
     </plugin>
   </gazebo>
-  <!-- Plugin LIDAR LD14P (simulado como RPLidar 360°) -->
+  <!-- LIDAR -->
   <gazebo reference="lidar_link">
     <sensor name="lidar" type="ray">
@@ -458,5 +437,5 @@
     </sensor>
   </gazebo>
-  <!-- Plugin Cámara RGB (AstraPro - canal color) -->
+  <!-- Cámara RGB -->
   <gazebo reference="camera_link">
     <sensor name="camera_rgb" type="camera">
@@ -471,8 +450,5 @@
           <format>R8G8B8</format>
         </image>
-        <clip>
-          <near>0.05</near>
-          <far>10.0</far>
-        </clip>
+        <clip><near>0.05</near><far>10.0</far></clip>
         <noise>
           <type>gaussian</type>
@@ -490,5 +466,4 @@
       </plugin>
     </sensor>
-    <!-- Plugin Profundidad (AstraPro - canal depth) -->
     <sensor name="camera_depth" type="depth">
       <always_on>true</always_on>
@@ -496,12 +471,6 @@
       <camera>
         <horizontal_fov>1.089</horizontal_fov>
-        <image>
-          <width>640</width>
-          <height>480</height>
-        </image>
-        <clip>
-          <near>0.1</near>
-          <far>8.0</far>
-        </clip>
+        <image><width>640</width><height>480</height></image>
+        <clip><near>0.1</near><far>8.0</far></clip>
       </camera>
       <plugin name="depth_plugin" filename="libgazebo_ros_camera.so">
@@ -516,5 +485,5 @@
     </sensor>
   </gazebo>
-  <!-- Plugin IMU (SensorTile) -->
+  <!-- IMU -->
   <gazebo reference="base_link">
     <gravity>true</gravity>
@@ -544,22 +513,29 @@
     </sensor>
   </gazebo>
-  <!-- Material orugas -->
+  <!-- ============================================================
+       MATERIALES Y FRICCIÓN
+       Orugas visuales (sin contacto físico, solo apariencia)
+       Ruedas con fricción REALISTA (mu=0.8) y contacto menos rígido
+       ============================================================ -->
   <gazebo reference="track_left">
-    <mu1>0.9</mu1><mu2>0.9</mu2>
     <material>Gazebo/Black</material>
   </gazebo>
   <gazebo reference="track_right">
-    <mu1>0.9</mu1><mu2>0.9</mu2>
     <material>Gazebo/Black</material>
   </gazebo>
-  <!-- Fricción ruedas sobre arena -->
   <gazebo reference="wheel_left">
-    <mu1>1.5</mu1><mu2>1.5</mu2>
-    <kp>500000</kp><kd>10</kd>
+    <mu1>0.8</mu1>
+    <mu2>0.8</mu2>
+    <kp>100000</kp>
+    <kd>10</kd>
+    <fdir1>1 0 0</fdir1>
     <material>Gazebo/Black</material>
   </gazebo>
   <gazebo reference="wheel_right">
-    <mu1>1.5</mu1><mu2>1.5</mu2>
-    <kp>500000</kp><kd>10</kd>
+    <mu1>0.8</mu1>
+    <mu2>0.8</mu2>
+    <kp>100000</kp>
+    <kd>10</kd>
+    <fdir1>1 0 0</fdir1>
     <material>Gazebo/Black</material>
   </gazebo>
